Commit message: 更新260/270/280/320/p340/myarm/mybuddy urdf模型关节运动范围

File: mycobot_description/urdf/mycobot_280_jn/mycobot_280_jn.urdf (robot description, URDF)
Before this commit: robot firefighter, 7 links, 6 joints
Joints:
- joint joint2_to_joint1: limit lower=-3.14 upper=3.14159 effort=1000.0 velocity=0 -> lower=-2.9322 upper=2.9322 effort=1000.0 velocity=0
- joint joint3_to_joint2: limit lower=-3.14 upper=3.14159 effort=1000.0 velocity=0 -> lower=-2.3562 upper=2.3562 effort=1000.0 velocity=0
- joint joint4_to_joint3: limit lower=-3.14 upper=3.14159 effort=1000.0 velocity=0 -> lower=-2.618 upper=2.618 effort=1000.0 velocity=0
- joint joint5_to_joint4: limit lower=-3.14 upper=3.14159 effort=1000.0 velocity=0 -> lower=-2.5307 upper=2.5307 effort=1000.0 velocity=0
- joint joint6_to_joint5: limit lower=-3.14 upper=3.14159 effort=1000.0 velocity=0 -> lower=-2.8798 upper=2.8798 effort=1000.0 velocity=0
- joint joint6output_to_joint6: limit lower=-3.14 upper=3.14159 effort=1000.0 velocity=0 -> lower=-3.14159 upper=3.14159 effort=1000.0 velocity=0

File: mycobot_description/urdf/mycobot_280_m5/mycobot_280_m5.urdf (robot description, URDF)
Before this commit: robot firefighter, 8 links, 7 joints
Joints:
- joint joint2_to_joint1: limit lower=-3.14 upper=3.14159 effort=1000.0 velocity=0 -> lower=-2.9322 upper=2.9322 effort=1000.0 velocity=0
- joint joint3_to_joint2: limit lower=-3.14 upper=3.14159 effort=1000.0 velocity=0 -> lower=-2.3562 upper=2.3562 effort=1000.0 velocity=0
- joint joint4_to_joint3: limit lower=-3.14 upper=3.14159 effort=1000.0 velocity=0 -> lower=-2.618 upper=2.618 effort=1000.0 velocity=0
- joint joint5_to_joint4: limit lower=-3.14 upper=3.14159 effort=1000.0 velocity=0 -> lower=-2.5307 upper=2.5307 effort=1000.0 velocity=0
- joint joint6_to_joint5: limit lower=-3.14 upper=3.14159 effort=1000.0 velocity=0 -> lower=-2.8798 upper=2.8798 effort=1000.0 velocity=0
- joint joint6output_to_joint6: limit lower=-3.14 upper=3.14159 effort=1000.0 velocity=0 -> lower=-3.14159 upper=3.14159 effort=1000.0 velocity=0

File: mycobot_description/urdf/mycobot_280_m5/mycobot_280_m5_with_camera_flange.urdf (robot description, URDF)
Before this commit: robot firefighter, 9 links, 8 joints
Joints:
- joint joint2_to_joint1: limit lower=-2.879793 upper=2.879793 effort=1000.0 velocity=0 -> lower=-2.9322 upper=2.9322 effort=1000.0 velocity=0
- joint joint3_to_joint2: limit lower=-2.879793 upper=2.879793 effort=1000.0 velocity=0 -> lower=-2.3562 upper=2.3562 effort=1000.0 velocity=0
- joint joint4_to_joint3: limit lower=-2.879793 upper=2.879793 effort=1000.0 velocity=0 -> lower=-2.618 upper=2.618 effort=1000.0 velocity=0
- joint joint5_to_joint4: limit lower=-2.879793 upper=2.879793 effort=1000.0 velocity=0 -> lower=-2.5307 upper=2.5307 effort=1000.0 velocity=0
- joint joint6_to_joint5: limit lower=-2.879793 upper=2.879793 effort=1000.0 velocity=0 -> lower=-2.8798 upper=2.8798 effort=1000.0 velocity=0
- joint joint6output_to_joint6: limit lower=-3.05 upper=3.05 effort=1000.0 velocity=0 -> lower=-3.14159 upper=3.14159 effort=1000.0 velocity=0

File: mycobot_description/urdf/mycobot_280_m5/mycobot_280_m5_with_camera_flange_pump.urdf (robot description, URDF)
Before this commit: robot firefighter, 11 links, 10 joints
Joints:
- joint joint2_to_joint1: limit lower=-2.879793 upper=2.879793 effort=1000.0 velocity=0 -> lower=-2.9322 upper=2.9322 effort=1000.0 velocity=0
- joint joint3_to_joint2: limit lower=-2.879793 upper=2.879793 effort=1000.0 velocity=0 -> lower=-2.3562 upper=2.3562 effort=1000.0 velocity=0
- joint joint4_to_joint3: limit lower=-2.879793 upper=2.879793 effort=1000.0 velocity=0 -> lower=-2.618 upper=2.618 effort=1000.0 velocity=0
- joint joint5_to_joint4: limit lower=-2.879793 upper=2.879793 effort=1000.0 velocity=0 -> lower=-2.5307 upper=2.5307 effort=1000.0 velocity=0
- joint joint6_to_joint5: limit lower=-2.879793 upper=2.879793 effort=1000.0 velocity=0 -> lower=-2.8798 upper=2.8798 effort=1000.0 velocity=0
- joint joint6output_to_joint6: limit lower=-3.05 upper=3.05 effort=1000.0 velocity=0 -> lower=-3.14159 upper=3.14159 effort=1000.0 velocity=0

File: mycobot_description/urdf/mycobot_280_m5/mycobot_280_m5_with_pump.urdf (robot description, URDF)
Before this commit: robot firefighter, 10 links, 9 joints
Joints:
- joint joint2_to_joint1: limit lower=-2.879793 upper=2.879793 effort=1000.0 velocity=0 -> lower=-2.9322 upper=2.9322 effort=1000.0 velocity=0
- joint joint3_to_joint2: limit lower=-2.879793 upper=2.879793 effort=1000.0 velocity=0 -> lower=-2.3562 upper=2.3562 effort=1000.0 velocity=0
- joint joint4_to_joint3: limit lower=-2.879793 upper=2.879793 effort=1000.0 velocity=0 -> lower=-2.618 upper=2.618 effort=1000.0 velocity=0
- joint joint5_to_joint4: limit lower=-2.879793 upper=2.879793 effort=1000.0 velocity=0 -> lower=-2.5307 upper=2.5307 effort=1000.0 velocity=0
- joint joint6_to_joint5: limit lower=-2.879793 upper=2.879793 effort=1000.0 velocity=0 -> lower=-2.8798 upper=2.8798 effort=1000.0 velocity=0
- joint joint6output_to_joint6: limit lower=-3.05 upper=3.05 effort=1000.0 velocity=0 -> lower=-3.14159 upper=3.14159 effort=1000.0 velocity=0

File: mycobot_description/urdf/mycobot_280_m5/mycobot_with_vision.urdf (robot description, URDF)
Before this commit: robot mycobot_ai, 8 links, 7 joints
Joints:
- joint joint2_to_joint1: limit lower=-3.14 upper=3.14159 effort=1000.0 velocity=0 -> lower=-2.9322 upper=2.9322 effort=1000.0 velocity=0
- joint joint3_to_joint2: limit lower=-3.14 upper=3.14159 effort=1000.0 velocity=0 -> lower=-2.3562 upper=2.3562 effort=1000.0 velocity=0
- joint joint4_to_joint3: limit lower=-3.14 upper=3.14159 effort=1000.0 velocity=0 -> lower=-2.618 upper=2.618 effort=1000.0 velocity=0
- joint joint5_to_joint4: limit lower=-3.14 upper=3.14159 effort=1000.0 velocity=0 -> lower=-2.5307 upper=2.5307 effort=1000.0 velocity=0
- joint joint6_to_joint5: limit lower=-3.14 upper=3.14159 effort=1000.0 velocity=0 -> lower=-2.8798 upper=2.8798 effort=1000.0 velocity=0
- joint joint6output_to_joint6: limit lower=-3.14 upper=3.14159 effort=1000.0 velocity=0 -> lower=-3.14159 upper=3.14159 effort=1000.0 velocity=0

File: mycobot_description/urdf/mycobot_280_pi/mycobot_280_pi.urdf (robot description, URDF)
Before this commit: robot firefighter, 8 links, 7 joints
Joints:
- joint joint2_to_joint1: limit lower=-3.14 upper=3.14159 effort=1000.0 velocity=0 -> lower=-2.9322 upper=2.9322 effort=1000.0 velocity=0
- joint joint3_to_joint2: limit lower=-3.14 upper=3.14159 effort=1000.0 velocity=0 -> lower=-2.3562 upper=2.3562 effort=1000.0 velocity=0
- joint joint4_to_joint3: limit lower=-3.14 upper=3.14159 effort=1000.0 velocity=0 -> lower=-2.618 upper=2.618 effort=1000.0 velocity=0
- joint joint5_to_joint4: limit lower=-3.14 upper=3.14159 effort=1000.0 velocity=0 -> lower=-2.5307 upper=2.5307 effort=1000.0 velocity=0
- joint joint6_to_joint5: limit lower=-3.14 upper=3.14159 effort=1000.0 velocity=0 -> lower=-2.8798 upper=2.8798 effort=1000.0 velocity=0
- joint joint6output_to_joint6: limit lower=-3.14 upper=3.14159 effort=1000.0 velocity=0 -> lower=-3.14159 upper=3.14159 effort=1000.0 velocity=0

File: mycobot_description/urdf/mycobot_280_pi/mycobot_280_pi_with_camera_flange.urdf (robot description, URDF)
Before this commit: robot firefighter, 9 links, 8 joints
Joints:
- joint joint2_to_joint1: limit lower=-3.14 upper=3.14159 effort=1000.0 velocity=0 -> lower=-2.9322 upper=2.9322 effort=1000.0 velocity=0
- joint joint3_to_joint2: limit lower=-3.14 upper=3.14159 effort=1000.0 velocity=0 -> lower=-2.3562 upper=2.3562 effort=1000.0 velocity=0
- joint joint4_to_joint3: limit lower=-3.14 upper=3.14159 effort=1000.0 velocity=0 -> lower=-2.618 upper=2.618 effort=1000.0 velocity=0
- joint joint5_to_joint4: limit lower=-3.14 upper=3.14159 effort=1000.0 velocity=0 -> lower=-3.5307 upper=3.5307 effort=1000.0 velocity=0
- joint joint6_to_joint5: limit lower=-3.14 upper=3.14159 effort=1000.0 velocity=0 -> lower=-2.8798 upper=2.8798 effort=1000.0 velocity=0
- joint joint6output_to_joint6: limit lower=-3.14 upper=3.14159 effort=1000.0 velocity=0 -> lower=-3.14159 upper=3.14159 effort=1000.0 velocity=0

File: mycobot_description/urdf/mycobot_280_pi/mycobot_280_pi_with_camera_flange_pump.urdf (robot description, URDF)
Before this commit: robot firefighter, 11 links, 10 joints
Joints:
- joint joint2_to_joint1: limit lower=-3.14 upper=3.14159 effort=1000.0 velocity=0 -> lower=-2.9322 upper=2.9322 effort=1000.0 velocity=0
- joint joint3_to_joint2: limit lower=-3.14 upper=3.14159 effort=1000.0 velocity=0 -> lower=-2.3562 upper=2.3562 effort=1000.0 velocity=0
- joint joint4_to_joint3: limit lower=-3.14 upper=3.14159 effort=1000.0 velocity=0 -> lower=-2.618 upper=2.618 effort=1000.0 velocity=0
- joint joint5_to_joint4: limit lower=-3.14 upper=3.14159 effort=1000.0 velocity=0 -> lower=-2.5307 upper=2.5307 effort=1000.0 velocity=0
- joint joint6_to_joint5: limit lower=-3.14 upper=3.14159 effort=1000.0 velocity=0 -> lower=-2.8798 upper=2.8798 effort=1000.0 velocity=0
- joint joint6output_to_joint6: limit lower=-3.14 upper=3.14159 effort=1000.0 velocity=0 -> lower=-3.14159 upper=3.14159 effort=1000.0 velocity=0

File: mycobot_description/urdf/mycobot_280_pi/mycobot_280_pi_with_pump.urdf (robot description, URDF)
Before this commit: robot firefighter, 10 links, 9 joints
Joints:
- joint joint2_to_joint1: limit lower=-3.14 upper=3.14159 effort=1000.0 velocity=0 -> lower=-2.9322 upper=2.9322 effort=1000.0 velocity=0
- joint joint3_to_joint2: limit lower=-3.14 upper=3.14159 effort=1000.0 velocity=0 -> lower=-2.3562 upper=2.3562 effort=1000.0 velocity=0
- joint joint4_to_joint3: limit lower=-3.14 upper=3.14159 effort=1000.0 velocity=0 -> lower=-2.618 upper=2.618 effort=1000.0 velocity=0
- joint joint5_to_joint4: limit lower=-3.14 upper=3.14159 effort=1000.0 velocity=0 -> lower=-2.5307 upper=2.5307 effort=1000.0 velocity=0
- joint joint6_to_joint5: limit lower=-3.14 upper=3.14159 effort=1000.0 velocity=0 -> lower=-2.8798 upper=2.8798 effort=1000.0 velocity=0
- joint joint6output_to_joint6: limit lower=-3.14 upper=3.14159 effort=1000.0 velocity=0 -> lower=-3.14159 upper=3.14159 effort=1000.0 velocity=0

File: mycobot_description/urdf/mycobot_280_x3pi/mycobot_280_x3pi.urdf (robot description, URDF)
Before this commit: robot firefighter, 7 links, 6 joints
Joints:
- joint joint2_to_joint1: limit lower=-3.14 upper=3.14159 effort=1000.0 velocity=0 -> lower=-2.9322 upper=2.9322 effort=1000.0 velocity=0
- joint joint3_to_joint2: limit lower=-3.14 upper=3.14159 effort=1000.0 velocity=0 -> lower=-2.3562 upper=2.3562 effort=1000.0 velocity=0
- joint joint4_to_joint3: limit lower=-3.14 upper=3.14159 effort=1000.0 velocity=0 -> lower=-2.618 upper=2.618 effort=1000.0 velocity=0
- joint joint5_to_joint4: limit lower=-3.14 upper=3.14159 effort=1000.0 velocity=0 -> lower=-2.5307 upper=2.5307 effort=1000.0 velocity=0
- joint joint6_to_joint5: limit lower=-3.14 upper=3.14159 effort=1000.0 velocity=0 -> lower=-2.8798 upper=2.8798 effort=1000.0 velocity=0
- joint joint6output_to_joint6: limit lower=-3.14 upper=3.14159 effort=1000.0 velocity=0 -> lower=-3.14159 upper=3.14159 effort=1000.0 velocity=0

File: mycobot_description/urdf/mycobot_280_x5pi/mycobot_280_x5pi.urdf (robot description, URDF)
Before this commit: robot firefighter, 7 links, 6 joints
Joints:
- joint joint2_to_joint1: limit lower=-2.93 upper=2.93 effort=1000.0 velocity=0 -> lower=-2.9322 upper=2.9322 effort=1000.0 velocity=0
- joint joint3_to_joint2: limit lower=-2.35 upper=2.35 effort=1000.0 velocity=0 -> lower=-2.3562 upper=2.3562 effort=1000.0 velocity=0
- joint joint4_to_joint3: limit lower=-2.61 upper=2.61 effort=1000.0 velocity=0 -> lower=-2.618 upper=2.618 effort=1000.0 velocity=0
- joint joint5_to_joint4: limit lower=-2.53 upper=2.53 effort=1000.0 velocity=0 -> lower=-2.5307 upper=2.5307 effort=1000.0 velocity=0
- joint joint6_to_joint5: limit lower=-2.87 upper=2.87 effort=1000.0 velocity=0 -> lower=-2.8798 upper=2.8798 effort=1000.0 velocity=0
- joint joint6output_to_joint6: limit lower=-3.14 upper=3.14 effort=1000.0 velocity=0 -> lower=-3.14159 upper=3.14159 effort=1000.0 velocity=0

File: mycobot_description/urdf/mycobot_320_m5_2022/mycobot_320_m5_2022.urdf (robot description, URDF)
Before this commit: robot firefighter, 7 links, 6 joints
Joints:
- joint joint2_to_joint1: limit lower=-2.87 upper=2.87 effort=1000.0 velocity=0 -> lower=-2.9321 upper=2.9321 effort=1000.0 velocity=0
- joint joint3_to_joint2: limit lower=-2.879 upper=2.879 effort=1000.0 velocity=0 -> lower=-2.3561 upper=2.3561 effort=1000.0 velocity=0
- joint joint4_to_joint3: limit lower=-2.879 upper=2.879 effort=1000.0 velocity=0 -> lower=-2.5307 upper=2.5307 effort=1000.0 velocity=0
- joint joint5_to_joint4: limit lower=-2.879 upper=2.879 effort=1000.0 velocity=0 -> lower=-2.5830 upper=2.5830 effort=1000.0 velocity=0
- joint joint6_to_joint5: limit lower=-2.879 upper=2.879 effort=1000.0 velocity=0 -> lower=-2.9321 upper=2.9321 effort=1000.0 velocity=0
- joint joint6output_to_joint6: limit lower=-3.05 upper=3.05 effort=1000.0 velocity=0 -> lower=-3.14159 upper=3.14159 effort=1000.0 velocity=0

File: mycobot_description/urdf/mycobot_320_pi_2022/mycobot_320_pi_2022.urdf (robot description, URDF)
Before this commit: robot firefighter, 7 links, 6 joints
Joints:
- joint joint2_to_joint1: limit lower=-2.96 upper=2.96 effort=1000.0 velocity=0 -> lower=-2.9321 upper=2.9321 effort=1000.0 velocity=0
- joint joint3_to_joint2: limit lower=-2.79 upper=2.79 effort=1000.0 velocity=0 -> lower=-2.3561 upper=2.3561 effort=1000.0 velocity=0
- joint joint4_to_joint3: limit lower=-2.79 upper=2.79 effort=1000.0 velocity=0 -> lower=-2.5307 upper=2.5307 effort=1000.0 velocity=0
- joint joint5_to_joint4: limit lower=-2.79 upper=2.79 effort=1000.0 velocity=0 -> lower=-2.5830 upper=2.5830 effort=1000.0 velocity=0
- joint joint6_to_joint5: limit lower=-2.96 upper=2.96 effort=1000.0 velocity=0 -> lower=-2.9321 upper=2.9321 effort=1000.0 velocity=0
- joint joint6output_to_joint6: limit lower=-3.05 upper=3.05 effort=1000.0 velocity=0 -> lower=-3.14159 upper=3.14159 effort=1000.0 velocity=0

File: mycobot_description/urdf/mypalletizer_260_m5/mypalletizer_260_m5.urdf (robot description, URDF)
Before this commit: robot firefighter, 6 links, 5 joints
Links:
- link base: geometry collision mesh filename=package://mycobot_description/urdf/mypalletizer_260_m5/base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; visual mesh filename=package://mycobot_description/urdf/mypalletizer_260_m5/base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
- link link1: geometry collision mesh filename=package://mycobot_description/urdf/mypalletizer_260_m5/link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; visual mesh filename=package://mycobot_description/urdf/mypalletizer_260_m5/link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
- link link2: geometry collision mesh filename=package://mycobot_description/urdf/mypalletizer_260_m5/link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; visual mesh filename=package://mycobot_description/urdf/mypalletizer_260_m5/link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
- link link3: geometry collision mesh filename=package://mycobot_description/urdf/mypalletizer_260_m5/link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; visual mesh filename=package://mycobot_description/urdf/mypalletizer_260_m5/link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
- link link4: geometry collision mesh filename=package://mycobot_description/urdf/mypalletizer_260_m5/link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; visual mesh filename=package://mycobot_description/urdf/mypalletizer_260_m5/link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
Joints:
- joint joint2_to_joint1: limit lower=-0.014 upper=1.49 effort=1000.0 velocity=0 -> lower=-0.0349 upper=1.5708 effort=1000.0 velocity=0
- joint joint3_to_joint2: limit lower=-0.213 upper=0.872665 effort=1000.0 velocity=0 -> lower=-1.6057 upper=1.0471 effort=1000.0 velocity=0

File: mycobot_description/urdf/mypalletizer_260_pi/mypalletizer_260_pi.urdf (robot description, URDF)
Before this commit: robot firefighter, 6 links, 5 joints
Links:
- link base: geometry collision mesh filename=package://mycobot_description/urdf/mypalletizer_260_pi/base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; visual mesh filename=package://mycobot_description/urdf/mypalletizer_260_pi/base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
- link link1: geometry collision mesh filename=package://mycobot_description/urdf/mypalletizer_260_pi/link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; visual mesh filename=package://mycobot_description/urdf/mypalletizer_260_pi/link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
- link link2: geometry collision mesh filename=package://mycobot_description/urdf/mypalletizer_260_pi/link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; visual mesh filename=package://mycobot_description/urdf/mypalletizer_260_pi/link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
- link link3: geometry collision mesh filename=package://mycobot_description/urdf/mypalletizer_260_pi/link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; visual mesh filename=package://mycobot_description/urdf/mypalletizer_260_pi/link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
- link link4: geometry collision mesh filename=package://mycobot_description/urdf/mypalletizer_260_pi/link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; visual mesh filename=package://mycobot_description/urdf/mypalletizer_260_pi/link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
Joints:
- joint joint2_to_joint1: limit lower=-0.014 upper=1.49 effort=1000.0 velocity=0 -> lower=-0.0349 upper=1.5708 effort=1000.0 velocity=0
- joint joint3_to_joint2: limit lower=-0.213 upper=0.872665 effort=1000.0 velocity=0 -> lower=-1.6057 upper=1.0471 effort=1000.0 velocity=0

File: mycobot_description/urdf/mypalletizer_260_pi/mypalletizer_260_pi_aikit.urdf (robot description, URDF)
Before this commit: robot firefighter, 7 links, 6 joints
Links:
- link base: geometry collision mesh filename=package://mycobot_description/urdf/mypalletizer_260_pi/base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; visual mesh filename=package://mycobot_description/urdf/mypalletizer_260_pi/base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
- link env: geometry visual mesh filename=package://mycobot_description/urdf/mypalletizer_260_pi/suit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 scale=1.2 1.2 1.2
- link link1: geometry collision mesh filename=package://mycobot_description/urdf/mypalletizer_260_pi/link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; visual mesh filename=package://mycobot_description/urdf/mypalletizer_260_pi/link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
- link link2: geometry collision mesh filename=package://mycobot_description/urdf/mypalletizer_260_pi/link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; visual mesh filename=package://mycobot_description/urdf/mypalletizer_260_pi/link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
- link link3: geometry collision mesh filename=package://mycobot_description/urdf/mypalletizer_260_pi/link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; visual mesh filename=package://mycobot_description/urdf/mypalletizer_260_pi/link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
- link link4: geometry collision mesh filename=package://mycobot_description/urdf/mypalletizer_260_pi/link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; visual mesh filename=package://mycobot_description/urdf/mypalletizer_260_pi/link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
Joints:
- joint joint2_to_joint1: limit lower=-0.014 upper=1.49 effort=1000.0 velocity=0 -> lower=-0.0349 upper=1.5708 effort=1000.0 velocity=0
- joint joint3_to_joint2: limit lower=-0.213 upper=0.872665 effort=1000.0 velocity=0 -> lower=-1.6057 upper=1.0471 effort=1000.0 velocity=0

File: mycobot_description/urdf/ultraArm_p340/ultraArm_p340.urdf (robot description, URDF)
Before this commit: robot firefighter, 4 links, 3 joints
Joints:
- joint joint1_to_base: limit lower=-2.36 upper=2.967 effort=1000.0 velocity=0 -> lower=-2.6179 upper=2.967 effort=1000.0 velocity=0
- joint joint2_to_joint1: limit lower=0 upper=1.14 effort=1000.0 velocity=0 -> lower=-0.3490 upper=1.5708 effort=1000.0 velocity=0
- joint joint3_to_joint2: limit lower=0 upper=1.0472 effort=1000.0 velocity=0 -> lower=-0.0872 upper=1.9198 effort=1000.0 velocity=0
