Commit message: 更新600/630 URDF模型初始姿态

File: mycobot_description/urdf/mycobot_pro_600/mycobot_pro_600.urdf (robot description, URDF)
Before this commit: robot firefighter, 7 links, 6 joints
Joints:
- joint joint3_to_joint2: limit lower=-4.7123 upper=1.5708 effort=1000.0 velocity=0 -> lower=-3.14159 upper=3.14159 effort=1000.0 velocity=0; origin xyz=0 0  0 rpy=1.5708 0 0 -> xyz=0 0  0 rpy=1.5708 -1.5708 0
- joint joint5_to_joint4: limit lower=-4.5378 upper=1.3962 effort=1000.0 velocity=0 -> lower=-2.9670 upper=2.9670 effort=1000.0 velocity=0; origin xyz=0.25 0  -0.1091 rpy=0 0 0 -> xyz=0.25 0  -0.1091 rpy=0 0 1.5708

File: mycobot_description/urdf/mycobot_pro_630/mycobot_pro_630.urdf (robot description, URDF)
Before this commit: robot firefighter, 7 links, 6 joints
Joints:
- joint joint2_to_joint1: limit lower=-4.71 upper=1.5707 effort=1000.0 velocity=0 -> lower=-3.14159 upper=3.14159 effort=1000.0 velocity=0; origin xyz=0 0  0 rpy=1.5707 0 0 -> xyz=0 0  0 rpy=1.5707 -1.5708 0
- joint joint4_to_joint3: limit lower=-4.53 upper=1.3962 effort=1000.0 velocity=0 -> lower=-2.9670 upper=2.9670 effort=1000.0 velocity=0; origin xyz=0.267 0  -0.0745 rpy=0 0 0 -> xyz=0.267 0  -0.0745 rpy=0 0 1.5708
